File: Board/instrument_lowpass/instrument_lowpass.kicad_pcb (KiCad board)
At the start: 2 copper layers, 80 x 45 mm, 43 parts, among them J1 Conn_Coaxial, J2 Conn_Coaxial, U1 NJM2114, U2 INA849DGKR

Commit message: add board design§
Parts:
- TP1: value TP -> cutoff_signal+
- TP2: value TP -> cutoff_signal-
- TP3: value TP -> cutoff_reference-
- TP4: value TP -> cutoff_reference+
- TP5: value TP -> gain-
- TP7: value TP -> gain+
- moved TP7 44.7 mm to (109.9, 53.9)
- moved TP5 36.8 mm to (110.0, 57.6)
- moved R11 34.6 mm to (174.4, 60.6), turned to -90 degrees
- moved R12 33.2 mm to (174.7, 65.0), turned to 180 degrees
- moved TP1 20.9 mm to (113.1, 88.1)
- moved U1 20.7 mm to (162.2, 56.0)
- moved TP2 20.6 mm to (113.1, 92.0)
- moved C8 20.4 mm to (112.3, 74.2)
- moved C3 19.5 mm to (112.3, 67.5)
- moved TP3 19.4 mm to (109.5, 92.0)
- moved TP4 19.3 mm to (109.5, 88.0)
- moved U2 18.0 mm to (139.8, 73.2)
- moved R6 16.9 mm to (134.1, 73.2)
- moved R5 16.7 mm to (130.6, 73.2)
- moved TP11 16.0 mm to (169.5, 78.7)
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Routing:
- net Net-(C1-Pad2): track 0.00 -> 89.4 mm
- net +9V: track 0.00 -> 69.0 mm
- net Net-(C13-Pad2): track 0.00 -> 68.3 mm
- net -9V: track 0.00 -> 50.7 mm
- net Net-(C10-Pad2): track 0.00 -> 48.2 mm, vias 0 -> 2
- net Net-(R6-Pad1): track 0.00 -> 39.1 mm, vias 0 -> 1
- net /input: track 0.00 -> 36.7 mm
- net Net-(J2-Pad1): track 0.00 -> 35.8 mm
- net Net-(C13-Pad1): track 0.00 -> 35.5 mm
- net Net-(C10-Pad1): track 0.00 -> 31.4 mm
- net Net-(R5-Pad1): track 0.00 -> 30.2 mm, vias 0 -> 1
- net Net-(R3-Pad2): track 0.00 -> 28.9 mm, vias 0 -> 1
- net Net-(R4-Pad1): track 0.00 -> 26.0 mm, vias 0 -> 1
- net Net-(R7-Pad1): track 0.00 -> 24.7 mm
- net Net-(R5-Pad2): track 0.00 -> 7.28 mm
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- added copper zone on B.Cu, net GND
- added copper zone on F.Cu, net GND

Commit message: move stuff on input side
Parts:
- moved R3 10.0 mm to (134.3, 63.2)
- moved C12 10.0 mm to (124.0, 62.2)
- moved C13 10.0 mm to (123.7, 83.0)
- moved C2 10.0 mm to (114.7, 63.0)
- moved C3 10.0 mm to (122.3, 67.3)
- moved C4 10.0 mm to (122.3, 70.8)
- moved C6 10.0 mm to (114.7, 82.0)
- moved C7 10.0 mm to (122.3, 77.1)
- moved C8 10.0 mm to (122.3, 74.0)
- moved R1 10.0 mm to (130.4, 63.2)
- moved R2 10.0 mm to (130.5, 81.8)
- moved R4 10.0 mm to (134.5, 81.8)
- moved R5 10.0 mm to (140.6, 73.0)
- moved R6 10.0 mm to (144.1, 73.0)
- moved U2 10.0 mm to (149.8, 73.0)
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Routing:
- net Net-(C13-Pad1): track 35.5 -> 58.0 mm
- net Net-(J2-Pad1): track 35.8 -> 25.7 mm
- net -9V: track 50.7 -> 40.6 mm
- net +9V: track 69.0 -> 59.1 mm
- net Net-(R6-Pad1): track 39.1 -> 48.5 mm
- net Net-(R5-Pad1): track 30.2 -> 39.6 mm
- net Net-(R3-Pad2): track 28.9 -> 38.1 mm
- net /input: track 36.7 -> 44.9 mm
- net Net-(R4-Pad1): track 26.0 -> 33.3 mm
- net Net-(C1-Pad2): track 89.4 -> 95.8 mm
- net Net-(C13-Pad2): track 68.3 -> 72.8 mm
- net GND: vias 0 -> 53
